File: pcb/Edifier_Remote/Edifier_Remote.sch (KiCad schematic (older format))
At the start: 4 parts, among them Q1 Q_NPN_BCE

Commit message: replace w/ esp 32 doit
Parts:
- removed ESP32: ESP32-DEVKITC-32D, MODULE_ESP32-DEVKITC-32D, symbol ESP32-DEVKITC-32D:ESP32-DEVKITC-32D
- added ESP32?: ESP32_Devkit_DOIT_V1, ESP32:ESP32_Devkit_DOIT_V1, symbol ESP32_Shield:ESP32_Devkit_DOIT_V1
Changed lines of the file:
@@
 EESchema Schematic File Version 4
+LIBS:Edifier_Remote-cache
 EELAYER 29 0
 EELAYER END
@@
 Comment4 ""
 $EndDescr
-$Comp
-L ESP32-DEVKITC-32D:ESP32-DEVKITC-32D ESP32
-U 1 1 5D48620E
-P 7500 3975
-F 0 "ESP32" H 7500 5142 50  0000 C CNN
-F 1 "ESP32-DEVKITC-32D" H 7500 5051 50  0000 C CNN
-F 2 "MODULE_ESP32-DEVKITC-32D" H 7500 3975 50  0001 L BNN
-F 3 "" H 7500 3975 50  0001 L BNN
-F 4 "None" H 7500 3975 50  0001 L BNN "Field4"
-F 5 "Unavailable" H 7500 3975 50  0001 L BNN "Field5"
-F 6 "ESP32-DEVKITC-32D" H 7500 3975 50  0001 L BNN "Field6"
-F 7 "None" H 7500 3975 50  0001 L BNN "Field7"
-F 8 "EVAL BOARD FOR ESP-WROOM-32" H 7500 3975 50  0001 L BNN "Field8"
-	1    7500 3975
-	1    0    0    -1
-$EndComp
 $Comp
 L Device:Q_NPN_BCE Q1
@@
 Text Label 6550 4275 0    50   ~ 0
 SEND
+$Comp
+L ESP32_Shield:ESP32_Devkit_DOIT_V1 ESP32?
+U 1 1 5D4BEDDD
+P 7425 4125
+F 0 "ESP32?" H 7425 5087 60  0000 C CNN
+F 1 "ESP32_Devkit_DOIT_V1" H 7425 4981 60  0000 C CNN
+F 2 "ESP32:ESP32_Devkit_DOIT_V1" H 7425 4125 60  0001 C CNN
+F 3 "" H 7425 4125 60  0001 C CNN
+	1    7425 4125
+	1    0    0    -1
+$EndComp
 $EndSCHEMATC

Commit message: update wires
Parts:
- gave numbers to parts that had none: 1
Changed lines of the file:
@@
 L power:GND #PWR0103
 U 1 1 5D49C889
-P 6425 4500
-F 0 "#PWR0103" H 6425 4250 50  0001 C CNN
-F 1 "GND" H 6430 4327 50  0000 C CNN
-F 2 "" H 6425 4500 50  0001 C CNN
-F 3 "" H 6425 4500 50  0001 C CNN
-	1    6425 4500
+P 6375 4900
+F 0 "#PWR0103" H 6375 4650 50  0001 C CNN
+F 1 "GND" H 6380 4727 50  0000 C CNN
+F 2 "" H 6375 4900 50  0001 C CNN
+F 3 "" H 6375 4900 50  0001 C CNN
+	1    6375 4900
 	1    0    0    -1
 $EndComp
 Wire Wire Line
-	6700 4375 6425 4375
-Wire Wire Line
-	6425 4375 6425 4500
-Wire Wire Line
-	6700 3075 6575 3075
-Text Label 6575 3075 0    50   ~ 0
-3V3
+	6375 4775 6375 4900
 Wire Wire Line
 	5275 4650 5500 4650
@@
 Text Label 5500 4850 0    50   ~ 0
 RECV
-Wire Wire Line
-	6700 4475 6550 4475
-Text Label 6550 4475 0    50   ~ 0
-RECV
-Wire Wire Line
-	6700 4275 6550 4275
-Text Label 6550 4275 0    50   ~ 0
-SEND
 $Comp
-L ESP32_Shield:ESP32_Devkit_DOIT_V1 ESP32?
+L ESP32_Shield:ESP32_Devkit_DOIT_V1 ESP32
 U 1 1 5D4BEDDD
 P 7425 4125
-F 0 "ESP32?" H 7425 5087 60  0000 C CNN
+F 0 "ESP32" H 7425 5087 60  0000 C CNN
 F 1 "ESP32_Devkit_DOIT_V1" H 7425 4981 60  0000 C CNN
 F 2 "ESP32:ESP32_Devkit_DOIT_V1" H 7425 4125 60  0001 C CNN
@@
 	1    0    0    -1
 $EndComp
+Wire Wire Line
+	6700 4775 6375 4775
+Wire Wire Line
+	6700 4575 6425 4575
+Wire Wire Line
+	6700 4675 6425 4675
+Text Label 6425 4575 0    50   ~ 0
+SEND
+Text Label 6425 4675 0    50   ~ 0
+RECV
+Wire Wire Line
+	8150 4875 8350 4875
+Text Label 8350 4875 0    50   ~ 0
+3V3
 $EndSCHEMATC
