File: pcb/Edifier_Remote/Edifier_Remote.sch (KiCad schematic (older format))
At the start: 4 parts, among them Q1 Q_NPN_BCE, U1 ESP32_DevKit

Commit message: finished board design
Parts:
- U1: footprint (none) -> ESP32:ESP32_DevKit_36PIN
Connections:
- net 3V3: now also U1.36 (3V3)
Changed lines of the file:
@@
 EESchema Schematic File Version 4
-EELAYER 26 0
+LIBS:Edifier_Remote-cache
+EELAYER 29 0
 EELAYER END
 $Descr A4 11693 8268
@@
 F 0 "U1" H 7750 5400 50  0000 C CNN
 F 1 "ESP32_DevKit" H 7750 5309 50  0000 C CNN
-F 2 "" H 7600 4625 50  0001 C CNN
+F 2 "ESP32:ESP32_DevKit_36PIN" H 7800 3350 50  0000 C CNN
 F 3 "" H 7600 4625 50  0001 C CNN
 	1    7800 4275
@@
 	6650 4975 6650 5250
 $Comp
-L power:GND #PWR?
+L power:GND #PWR0103
 U 1 1 5D4C572D
 P 6650 5250
-F 0 "#PWR?" H 6650 5000 50  0001 C CNN
+F 0 "#PWR0103" H 6650 5000 50  0001 C CNN
 F 1 "GND" H 6655 5077 50  0000 C CNN
 F 2 "" H 6650 5250 50  0001 C CNN
@@
 	1    0    0    -1
 $EndComp
+Wire Wire Line
+	8350 5075 8600 5075
+Text Label 8600 5075 0    50   ~ 0
+3V3
 $EndSCHEMATC
